File: carte alim V1.0.23.kicad_sch (KiCad schematic)
At the start: 16 parts, among them U1 B_Plug_5mm, U10 B_Plug_5mm, U11 B_Plug_5mm, U12 B_Plug_5mm, U2 XL4015, U3 YAAJ_DCDC_StepDown_LM2596, U4 YAAJ_DCDC_StepDown_LM2596, U5 YAAJ_DCDC_StepDown_LM2596, U6 B_Plug_5mm, U7 B_Plug_5mm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

Commit message: new carte
Parts:
- removed U6: B_Plug_5mm, Connector_Phoenix_MSTB:PhoenixContact_MSTBA_2,5_2-G-5,08_1x02_P5.08mm_Horizontal, symbol MSTB2,5_-5,08:B_Plug_5mm
- U2: footprint XL4015_converter:XL4015_Converter -> XL4015Footprint:XL4015_Converter
Connections:
- net GND: no longer U7.2
- net at R1.1, U1.2, U3.1 (Vin)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: now also U7.1
- net at F4.1, U2.1 (IN+): now also U7.2; no longer U7.1
Other:
- moved on the sheet: F4, U7

Commit message: carte final V3
Parts:
- removed D1: LED, LED_THT:LED_D3.0mm, symbol Device:LED
- removed R1: R, Resistor_THT:R_Axial_DIN0207_L6.3mm_D2.5mm_P10.16mm_Horizontal, symbol Device:R
- removed U10, U11, U12 (x2), U7, U9: B_Plug_5mm, Connector_Phoenix_MSTB:PhoenixContact_MSTBA_2,5_2-G-5,08_1x02_P5.08mm_Horizontal, symbol MSTB2,5_-5,08:B_Plug_5mm
- removed U3: YAAJ_DCDC_StepDown_LM2596, Footprints:YAAJ_DCDC_StepDown_LM2596, symbol yaaj_dcdc_stepdown_lm2596:YAAJ_DCDC_StepDown_LM2596
- added H1, H2, H3: MountingHole, MountingHole:MountingHole_2.2mm_M2_ISO7380, symbol Mechanical:MountingHole
- added J1, J2: Conn_01x02, Connector_JST:JST_XH_B2B-XH-A_1x02_P2.50mm_Vertical, symbol Connector_Generic:Conn_01x02
- added J3: Conn_01x04, Connector_JST:JST_XH_B4B-XH-A_1x04_P2.50mm_Vertical, symbol Connector_Generic:Conn_01x04
- added U8: B_Plug_5mm, Connector_Phoenix_MSTB:PhoenixContact_MSTBA_2,5_2-G-5,08_1x02_P5.08mm_Horizontal, symbol MSTB2,5_-5,08:B_Plug_5mm
Connections:
- net GND: now also J1.2 (Pin_2), J2.2 (Pin_2), J3.3 (Pin_3), J3.4 (Pin_4)
- net at U1.2, U4.1 (Vin), U5.1 (Vin): now also U8.1
- net at U2.3 (OUT+): now also J3.1 (Pin_1), J3.2 (Pin_2)
- net at U5.4 (Vout): now also J2.1 (Pin_1)
- net at U4.4 (Vout): now also J1.1 (Pin_1)
- net at F4.1, U2.1 (IN+): now also U8.2
